File: midiori.kicad_sch (KiCad schematic)
At the start: 65 parts, among them J1 x68000_expansion, J2 Conn_ARM_JTAG_SWD_10, J3 AudioJack3, J4 RJ12, J5 AudioJack3, J6 J_PI_ZERO, J8 Waveblaster Connector, J9 AudioJack3, SW2 ROM, SW3 SYNTH, SW4 SS-10-23NPE, U1 74LCX07, U10 ICE40HX1K-VQ100, U11 TLV75533PDBV, U15 U_GY-PCM5102, U2 AT25SF081-SSHD-X, U3 TLV73312PDBV, U4 SN74LVC8T245DWR, U5 SN74LVC8T245DWR, U6 SN74LVC8T245DWR, U7 SN74LVC8T245DWR, U8 SN74LVC8T245DWR, U9 SN74LVC8T245DWR, X1 16MHz

Commit message: Development board
Parts:
- removed SW4: SS-10-23NPE, SS-10-23NPE:SS1023NPE, symbol SS-10-23NPE:SS-10-23NPE
- removed U15: U_GY-PCM5102, llama:U_GY-PCM5102, symbol llama:U_GY-PCM5102
- added C24: 0.1uF, Capacitor_SMD:C_0805_2012Metric, symbol Device:C
- added C25, C26, C33, C34: 47uF, Capacitor_SMD:C_Elec_6.3x5.8, symbol Device:C_Polarized
- added C27, C35, C36: 5.6nF, Capacitor_SMD:C_0805_2012Metric, symbol Device:C
- added C31, C32: 10nF, Capacitor_SMD:C_0805_2012Metric, symbol Device:C
- added J10: AudioJack3, Connector_Audio:Jack_3.5mm_CUI_SJ1-3535NG_Horizontal, symbol Connector_Audio:AudioJack3
- added J11: PCM1802_board, Audio_Module:PCM1808_board, symbol Audio:PCM1802_board
- added J12: Conn_01x03_Pin, Connector_PinHeader_2.54mm:PinHeader_1x03_P2.54mm_Horizontal, symbol Connector:Conn_01x03_Pin
- added J7: AMP2, Audio_Module:AMP2_TH, symbol AMP2:AMP2
- added JP2, JP3, JP4: Jumper_3_Open, Jumper:SolderJumper-3_P1.3mm_Open_RoundedPad1.0x1.5mm, symbol Jumper:Jumper_3_Open
- added R1, R2: 18k, Resistor_SMD:R_0805_2012Metric, symbol Device:R
- added R12, R13: 560, Resistor_SMD:R_0805_2012Metric, symbol Device:R
- added SW1: RotaryEncoder_Switch, Rotary_Encoder:RotaryEncoder_Bourns_Horizontal_PEC09-2xxxF-Sxxxx, symbol Device:RotaryEncoder_Switch
- added X2: 12.288MHz, Oscillator:Oscillator_SMD_SeikoEpson_SG8002CA-4Pin_7.0x5.0mm, symbol Oscillator:SG-8002CA
- C28: value 0.1uF -> 5.6nF
- R10, R11, R7, R8: value 47k -> 10k; footprint Resistor_SMD:R_0805_2012Metric_Pad1.20x1.40mm_HandSolder -> Resistor_SMD:R_0805_2012Metric
- R4, R5: value 47k -> 560; footprint Resistor_SMD:R_0805_2012Metric_Pad1.20x1.40mm_HandSolder -> Resistor_SMD:R_0805_2012Metric
Connections:
- net L_Lo is gone; now on net +3V3: R8.1
- net +3V3: now also R11.1, C24.2, J11.12 (3V3), J11.5 (3V3), JP2.3 (B), JP3.3 (B), JP4.3 (B), X2.1 (OE), X2.4 (Vcc)
- net +5V: now also J11.6 (5V), J7.B20 (VIN); no longer C28.2
- net AGND: now also C28.2, C27.1, C35.1, C36.2, J10.S, J11.14 (GND), J12.2 (Pin_2), J7.A18 (GND), J7.A2 (GND), J7.A4 (GND); no longer R11.1, R7.1
- net GND: now also C24.1, C31.1, C32.1, J11.11 (GND), J11.4 (GND), J7.B1 (GND), J7.B11 (GND), J7.B13 (GND), J7.B15 (GND), J7.B17 (GND), J7.B19 (GND), J7.B3 (GND), J7.B5 (GND), J7.B7 (GND), J7.B9 (GND), JP2.1 (A), JP3.1 (A), JP4.1 (A), SW1.C, SW1.S2, X2.2 (GND); no longer C28.1
- net WT_L: now also J10.T, J11.13 (LIN)
- net WT_R: now also J10.R, J11.15 (RIN)
- net exreset: now also J7.A9 (/RESET)
- net mix_pwm: now reaches U10.82 (IOT_78)
- net mix_pwm: now also J7.A11 (MP2)
- net mix_d0: now reaches U10.83 (IOT_79)
- net mix_d0: now also J7.A13 (MP3)
- net mix_d1: now reaches U10.86 (IOT_81)
- net mix_d1: now also J7.A15 (MP8)
- net mix_d2: now reaches U10.89 (IOT_84_GBIN1)
- net mix_d2: now also J7.A17 (MP9)
- net I2S_BCK renamed bclk
- net bclk: now also J11.7 (BCK), J7.B16 (MP5)
- net I2S_DIN renamed sdata_pi
- net sdata_pi: now also J7.B14 (MP1)
- net I2S_LCK renamed lrclk
- net lrclk: now also J11.9 (LRC), J7.B18 (MP4)
- net LEFT renamed LEFT_OUT
- net LEFT_OUT: now also R4.2, C27.2
- removed net L_Hi: J9.T, R10.2, R11.2
- net L_Med: no longer names the net of R8.2
- net L_Med: now also R7.2, SW1.A; no longer R10.1
- net RIGHT renamed RIGHT_OUT
- net RIGHT_OUT: now also C28.1, R5.2
- removed net R_Hi: J9.R, R5.2, R7.2
- net R_Lo: no longer names the net of R4.1
- net R_Lo: now also C25.2
- net R_Med: no longer names the net of R5.1
- net R_Med: now also C26.2; no longer R4.2
- new net: C26.1, J7.A12 (DAC1)
- new net: J11.1 (Pin_1), JP2.2 (C)
- new net: J11.2 (MD1), JP3.2 (C)
- new net: J11.3 (MD0), JP4.2 (C)
- new net: C34.2, R13.1
- new net: J7.A1 (AD0), R1.2
- new net: J7.A3 (AD1), R2.2
- new net: R10.1, R11.2, SW1.B
- new net: C33.1, J7.A14 (DAC2)
- new net: C33.2, R12.1
- new net: C34.1, J7.A16 (DAC3)
- new net: C25.1, J7.A10 (DAC0)
- new net ADC0_L: J9.T, R1.1
- new net ADC0_R: J9.R, R2.1
- new net SEC_LEFT_OUT: C35.2, J12.3 (Pin_3), R12.2
- new net SEC_RIGHT_OUT: C36.1, J12.1 (Pin_1), R13.2
- new net mclk: J11.10 (SCK), J7.B2 (MCLK), X2.3 (OUT)
- new net mix_wb: J7.A6 (WB)
- new net rot_a: C31.2, J7.B8 (MP6), R7.1
- new net rot_b: C32.2, J7.B10 (MP7), R10.2
- new net rot_sw: J7.B6 (MP10), SW1.S1
- new net sdata_extadc: J11.8 (OUT), J7.B12 (MP0)
- no-connect marks 29 -> 34
Other:
- moved on the sheet: J5
